Commit message: edited urdf files

File: urdf/whisker_project.urdf (robot description, URDF)
Before this commit: robot whisker_project, 4 links, 3 joints
Links:
- added link world_link
Joints:
- added joint world_to_base: type fixed, parent world_link, child base_link, origin xyz=0 0 0 rpy=0 0 0

Commit message: Update whisker_project.urdf
Raised Lidar and Depth 5mm

File: urdf/whisker_project.urdf (robot description, URDF)
Before this commit: robot whisker_project, 5 links, 4 joints
Joints:
- joint depth_Joint: origin xyz=0.0600690949305007 0.0460822729755588 0.0341258110332986 rpy=0 0 0 -> xyz=0.0600690949305007 0.0460822729755588 0.0391258110332986 rpy=0 0 0
- joint lidar_Joint: origin xyz=-0.0423409050707997 -0.0300177645431443 0.0603652915318988 rpy=0 0 0 -> xyz=-0.0423409050707997 -0.0300177645431443 0.0653652915318988 rpy=0 0 0
