Commit message: apply fixes to urdf and csv for gsfm_description rename

File: urdf/gsfm_description.urdf (robot description, URDF)
Before this commit: robot whisker_project, 5 links, 4 joints
Links:
- link base_link: geometry collision mesh filename=package://gsfm_description/meshes/base_link.STL; visual mesh filename=package://gsfm_description/meshes/base_link.STL
- link depth_Link: geometry collision mesh filename=package://gsfm_description/meshes/depth_Link.STL; visual mesh filename=package://gsfm_description/meshes/depth_Link.STL
- link imu_Link: geometry collision mesh filename=package://gsfm_description/meshes/imu_Link.STL; visual mesh filename=package://gsfm_description/meshes/imu_Link.STL
- link lidar_Link: geometry collision mesh filename=package://gsfm_description/meshes/lidar_Link.STL; visual mesh filename=package://gsfm_description/meshes/lidar_Link.STL

Commit message: fix names of links

File: urdf/gsfm_description.urdf (robot description, URDF)
Before this commit: robot gsfm_description, 5 links, 4 joints
Links:
- removed link depth_Link
- removed link imu_Link
- removed link lidar_Link
- added link camera_link, mass 0.220446940128425; collision mesh filename=package://gsfm_description/meshes/camera_link.STL; visual mesh filename=package://gsfm_description/meshes/camera_link.STL
- added link imu_link, mass 0.943685156899018; collision mesh filename=package://gsfm_description/meshes/imu_link.STL; visual mesh filename=package://gsfm_description/meshes/imu_link.STL
- added link laser_link, mass 0.208750664901466; collision mesh filename=package://gsfm_description/meshes/laser_link.STL; visual mesh filename=package://gsfm_description/meshes/laser_link.STL
Joints:
- removed joint depth_Joint
- removed joint imu_Joint
- removed joint lidar_Joint
- added joint camera_joint: type fixed, parent base_link, child camera_link, origin xyz=0.0600690949305007 0.0460822729755588 0.039125811033298596 rpy=0 0 0, axis 0 0 0
- added joint imu_joint: type fixed, parent base_link, child imu_link, origin xyz=0.0215090949305007 0.0447830082299264 -0.0407741889667037 rpy=0 0 0, axis 0 0 0
- added joint laser_joint: type fixed, parent base_link, child laser_link, origin xyz=-0.0423409050707997 -0.0300177645431443 0.0653652915318988 rpy=0 0 0, axis 0 0 0
